File: PCB/Quarfinder rev2.brd (EAGLE design)
At the start: 44.4 x 81.3 mm, 41 parts, among them J1 TL32PO, X1 SMA-142-0711-821/826

Commit message: final pcb
Parts:
- moved J1 1.27 mm to (3.81, 7.62)
Routing:
- net RAWSWITCH: track 40.7 -> 42.6 mm
- net VIN: track 18.0 -> 18.5 mm
Changed lines of the file:
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@@
 <layer number="20" name="Dimension" color="24" fill="1" visible="yes" active="yes"/>
 <layer number="21" name="tPlace" color="7" fill="1" visible="yes" active="yes"/>
-<layer number="22" name="bPlace" color="7" fill="1" visible="yes" active="yes"/>
+<layer number="22" name="bPlace" color="7" fill="1" visible="no" active="yes"/>
 <layer number="23" name="tOrigins" color="15" fill="1" visible="yes" active="yes"/>
-<layer number="24" name="bOrigins" color="15" fill="1" visible="yes" active="yes"/>
+<layer number="24" name="bOrigins" color="15" fill="1" visible="no" active="yes"/>
 <layer number="25" name="tNames" color="7" fill="1" visible="yes" active="yes"/>
-<layer number="26" name="bNames" color="7" fill="1" visible="yes" active="yes"/>
+<layer number="26" name="bNames" color="7" fill="1" visible="no" active="yes"/>
 <layer number="27" name="tValues" color="7" fill="1" visible="no" active="yes"/>
 <layer number="28" name="bValues" color="7" fill="1" visible="no" active="yes"/>
@@
 <layer number="38" name="bTest" color="7" fill="1" visible="no" active="yes"/>
 <layer number="39" name="tKeepout" color="4" fill="11" visible="yes" active="yes"/>
-<layer number="40" name="bKeepout" color="1" fill="11" visible="yes" active="yes"/>
+<layer number="40" name="bKeepout" color="1" fill="11" visible="no" active="yes"/>
 <layer number="41" name="tRestrict" color="4" fill="10" visible="yes" active="yes"/>
-<layer number="42" name="bRestrict" color="1" fill="10" visible="yes" active="yes"/>
+<layer number="42" name="bRestrict" color="1" fill="10" visible="no" active="yes"/>
 <layer number="43" name="vRestrict" color="2" fill="10" visible="no" active="yes"/>
 <layer number="44" name="Drills" color="7" fill="1" visible="no" active="yes"/>
@@
 <layer number="50" name="dxf" color="7" fill="1" visible="no" active="no"/>
 <layer number="51" name="tDocu" color="7" fill="1" visible="yes" active="yes"/>
-<layer number="52" name="bDocu" color="7" fill="1" visible="yes" active="yes"/>
+<layer number="52" name="bDocu" color="7" fill="1" visible="no" active="yes"/>
 <layer number="53" name="tGND_GNDA" color="7" fill="9" visible="no" active="no"/>
 <layer number="54" name="bGND_GNDA" color="1" fill="9" visible="no" active="no"/>
@@
 <attribute name="VALUE" x="-3.81" y="26.3525" size="0.6096" layer="27" font="vector" ratio="20" rot="R180" align="top-center"/>
 </element>
-<element name="J1" library="switch" library_urn="urn:adsk.eagle:library:380" package="TL3XPO" package3d_urn="urn:adsk.eagle:package:27745/1" value="TL32PO" x="2.54" y="7.62" smashed="yes" rot="MR270">
-<attribute name="VALUE" x="7.62" y="12.7" size="1.778" layer="28" rot="MR270"/>
+<element name="J1" library="switch" library_urn="urn:adsk.eagle:library:380" package="TL3XPO" package3d_urn="urn:adsk.eagle:package:27745/1" value="TL32PO" x="3.81" y="7.62" smashed="yes" rot="MR270">
+<attribute name="VALUE" x="8.89" y="12.7" size="1.778" layer="28" rot="MR270"/>
 </element>
 <element name="R7" library="rcl" library_urn="urn:adsk.eagle:library:334" package="R1206" package3d_urn="urn:adsk.eagle:package:23540/2" value="" x="-3.81" y="-20.32" smashed="yes">
@@
 <contactref element="D2_R" pad="C"/>
 <contactref element="R8" pad="1"/>
-<via x="-24.13" y="-7.62" extent="1-16" drill="0.35"/>
-<via x="-22.86" y="-8.89" extent="1-16" drill="0.35"/>
+<via x="-24.13" y="-6.35" extent="1-16" drill="0.35"/>
+<via x="-22.86" y="-7.62" extent="1-16" drill="0.35"/>
+<via x="-21.59" y="-8.89" extent="1-16" drill="0.35"/>
 </signal>
 <signal name="N$8">
@@
 <wire x1="-2.9253" y1="-16.1588" x2="-2.786" y2="-16.2981" width="0.4064" layer="16"/>
 <wire x1="-2.9253" y1="-10.1689" x2="-2.9253" y2="-16.1588" width="0.4064" layer="16"/>
-<wire x1="4.8755" y1="-2.3681" x2="-2.9253" y2="-10.1689" width="0.4064" layer="16"/>
-<wire x1="4.8755" y1="8.2187" x2="4.8755" y2="-2.3681" width="0.4064" layer="16"/>
-<wire x1="3.0646" y1="10.0296" x2="4.8755" y2="8.2187" width="0.4064" layer="16"/>
-<wire x1="2.6467" y1="10.0296" x2="3.0646" y2="10.0296" width="0.4064" layer="16"/>
+<wire x1="6.1292" y1="-1.1144" x2="-2.9253" y2="-10.1689" width="0.4064" layer="16"/>
+<wire x1="6.1292" y1="8.358" x2="6.1292" y2="-1.1144" width="0.4064" layer="16"/>
+<wire x1="4.4576" y1="10.0296" x2="6.1292" y2="8.358" width="0.4064" layer="16"/>
+<wire x1="3.9004" y1="10.0296" x2="4.4576" y2="10.0296" width="0.4064" layer="16"/>
 <wire x1="-2.5074" y1="-20.1985" x2="-2.388" y2="-20.32" width="0.4064" layer="1"/>
-<wire x1="2.6467" y1="10.0296" x2="2.54" y2="10.16" width="0.4064" layer="16"/>
-<wire x1="1.1144" y1="11.4226" x2="-2.5074" y2="11.4226" width="0.4064" layer="16"/>
-<wire x1="2.3681" y1="10.1689" x2="1.1144" y2="11.4226" width="0.4064" layer="16"/>
+<wire x1="3.9004" y1="10.0296" x2="3.81" y2="10.16" width="0.4064" layer="16"/>
+<wire x1="2.3681" y1="11.4226" x2="-2.5074" y2="11.4226" width="0.4064" layer="16"/>
+<wire x1="3.6218" y1="10.1689" x2="2.3681" y2="11.4226" width="0.4064" layer="16"/>
 <wire x1="-2.5074" y1="11.4226" x2="-2.54" y2="11.43" width="0.4064" layer="16"/>
-<wire x1="2.3681" y1="10.1689" x2="2.54" y2="10.16" width="0.4064" layer="16"/>
+<wire x1="3.6218" y1="10.1689" x2="3.81" y2="10.16" width="0.4064" layer="16"/>
 <via x="-2.786" y="-18.5269" extent="1-16" drill="0.4064"/>
 </signal>
@@
 <contactref element="J1" pad="2"/>
 <wire x1="-6.2685" y1="-4.7362" x2="-6.2685" y2="-6.2685" width="0.4064" layer="16"/>
-<wire x1="0.1393" y1="1.6716" x2="-6.2685" y2="-4.7362" width="0.4064" layer="16"/>
-<wire x1="0.1393" y1="5.7113" x2="0.1393" y2="1.6716" width="0.4064" layer="16"/>
-<wire x1="1.9502" y1="7.5222" x2="0.1393" y2="5.7113" width="0.4064" layer="16"/>
-<wire x1="2.5074" y1="7.5222" x2="1.9502" y2="7.5222" width="0.4064" layer="16"/>
+<wire x1="1.393" y1="2.9253" x2="-6.2685" y2="-4.7362" width="0.4064" layer="16"/>
+<wire x1="1.393" y1="5.7113" x2="1.393" y2="2.9253" width="0.4064" layer="16"/>
+<wire x1="3.2039" y1="7.5222" x2="1.393" y2="5.7113" width="0.4064" layer="16"/>
+<wire x1="3.7611" y1="7.5222" x2="3.2039" y2="7.5222" width="0.4064" layer="16"/>
 <wire x1="-6.2685" y1="-6.2685" x2="-6.35" y2="-6.35" width="0.4064" layer="16"/>
-<wire x1="2.5074" y1="7.5222" x2="2.54" y2="7.62" width="0.4064" layer="16"/>
+<wire x1="3.7611" y1="7.5222" x2="3.81" y2="7.62" width="0.4064" layer="16"/>
 </signal>
 <signal name="N$16">
@@
 <contactref element="R6" pad="2"/>
 <wire x1="4.0397" y1="20.6164" x2="5.0148" y2="20.6164" width="0.254" layer="1"/>
-<wire x1="3.3432" y1="19.9199" x2="4.0397" y2="20.6164" width="0.254" layer="1"/>
-<wire x1="3.3432" y1="19.0841" x2="3.3432" y2="19.9199" width="0.254" layer="1"/>
-<wire x1="3.3432" y1="12.2584" x2="3.3432" y2="19.0841" width="0.254" layer="16"/>
-<wire x1="5.7113" y1="9.8903" x2="3.3432" y2="12.2584" width="0.254" layer="16"/>
-<wire x1="5.7113" y1="-32.3176" x2="5.7113" y2="9.8903" width="0.254" layer="16"/>
-<wire x1="-1.2537" y1="-39.2826" x2="5.7113" y2="-32.3176" width="0.254" layer="16"/>
+<wire x1="0.9751" y1="17.5518" x2="4.0397" y2="20.6164" width="0.254" layer="1"/>
+<wire x1="0.9751" y1="-3.6218" x2="0.9751" y2="17.5518" width="0.254" layer="1"/>
+<wire x1="3.0646" y1="-5.7113" x2="0.9751" y2="-3.6218" width="0.254" layer="1"/>
+<wire x1="3.0646" y1="-34.9643" x2="3.0646" y2="-5.7113" width="0.254" layer="16"/>
+<wire x1="-1.2537" y1="-39.2826" x2="3.0646" y2="-34.9643" width="0.254" layer="16"/>
 <wire x1="5.0148" y1="20.6164" x2="5.08" y2="20.74" width="0.254" layer="1"/>
 <wire x1="-1.2537" y1="-39.2826" x2="-1.27" y2="-39.37" width="0.254" layer="16"/>
-<via x="3.3432" y="19.0841" extent="1-16" drill="0.35"/>
+<via x="3.0646" y="-5.7113" extent="1-16" drill="0.35"/>
 </signal>
 <signal name="N$19">
